File: hw/baseline_project.kicad_sch (KiCad schematic)
At the start: 20 parts, among them J101 EXT_3V3, Q101 IRLD024PBF, SW101 UP, SW102 DOWN, SW103 LEFT, SW104 RIGHT, SW105 MODE, U101 EK-TM4C123GXL, U102 ESP8266-1, U103 Adafruit ST7735R

Commit message: tiny bit of prep
Parts:
- SW101: value UP -> MODE
- SW102: value DOWN -> LEFT
- SW103: value LEFT -> RIGHT
- SW104: value RIGHT -> UP
- SW105: value MODE -> DOWN
Connections:
- net PC4: no longer SW101.2
- net PC5: no longer SW104.2
- net PC6: no longer SW103.2
- net PC7: no longer SW102.2
- net PE0: now also SW101.2
- net PE1: now also SW102.2
- net PE2: now also SW103.2
- net PE3: now also SW104.2
- net PE4: now also SW105.2
- net PF4: no longer SW105.2
